Commit message: push

File: src/motoman/motoman_hc10_support/urdf/hc10.xacro (robot description, xacro)
@@ -1,5 +1,84 @@
 <?xml version="1.0" ?>
-<robot name="motoman_hc10" xmlns:xacro="http://ros.org/wiki/xacro">
+<robot name="motoman_hc10" xmlns:xacro="http://www.ros.org/wiki/xacro">
+  <!-- Include the HC10 macros -->
   <xacro:include filename="$(find motoman_hc10_support)/urdf/hc10_macro.xacro" />
   <xacro:motoman_hc10 prefix=""/>
+  <!-- ========================= -->
+  <!-- Attach HC10 to world -->
+  <!-- ========================= -->
+  <joint name="base_joint" type="fixed">
+    <parent link="world"/>
+    <child link="base_link"/>
+  </joint>
+  <!-- ========================= -->
+  <!-- Table (optional, for reference) -->
+  <!-- ========================= -->
+  <link name="table">
+    <visual>
+      <geometry>
+        <box size="1 0.5 0.05"/>
+      </geometry>
+      <material name="Brown"/>
+    </visual>
+  </link>
+  <joint name="table_joint" type="fixed">
+    <parent link="world"/>
+    <child link="table"/>
+    <origin xyz="0 0 0" rpy="0 0 0"/>
+  </joint>
+  <!-- ========================= -->
+  <!-- Attach Kinect Camera to HC10 tool -->
+  <!-- ========================= -->
+  <link name="camera_depth_frame">
+    <visual>
+      <geometry>
+        <box size="0.05 0.05 0.05"/>
+      </geometry>
+      <material name="Gray"/>
+    </visual>
+  </link>
+  <joint name="camera_tool_joint" type="fixed">
+    <parent link="tool0"/> <!-- HC10 tool flange -->
+    <child link="camera_depth_frame"/>
+    <origin xyz="0 0 0.01" rpy="0 0 0"/> <!-- adjust as needed -->
+  </joint>
+  <!-- ========================= -->
+  <!-- Gazebo sensor plugin -->
+  <!-- ========================= -->
+  <gazebo reference="camera_depth_frame">
+    <sensor name="kinect_camera" type="depth">
+      <update_rate>20</update_rate>
+      <camera>
+        <horizontal_fov>1.047198</horizontal_fov>
+        <image>
+          <width>640</width>
+          <height>480</height>
+          <format>B8G8R8</format>
+        </image>
+        <clip>
+          <near>0.05</near>
+          <far>3</far>
+        </clip>
+      </camera>
+      <plugin name="kinect_controller" filename="libgazebo_ros_openni_kinect.so">
+        <baseline>0.1</baseline>
+        <alwaysOn>true</alwaysOn>
+        <updateRate>10</updateRate>
+        <cameraName>camera_ir</cameraName>
+        <imageTopicName>/camera/color/image_raw</imageTopicName>
+        <cameraInfoTopicName>/camera/color/camera_info</cameraInfoTopicName>
+        <depthImageTopicName>/camera/depth/image_raw</depthImageTopicName>
+        <depthImageCameraInfoTopicName>/camera/depth/camera_info</depthImageCameraInfoTopicName>
+        <pointCloudTopicName>/camera/depth/points</pointCloudTopicName>
+        <frameName>camera_depth_optical_frame</frameName>
+        <distortion_k1>0.0</distortion_k1>
+        <distortion_k2>0.0</distortion_k2>
+        <distortion_k3>0.0</distortion_k3>
+        <distortion_t1>0.0</distortion_t1>
+        <distortion_t2>0.0</distortion_t2>
+        <pointCloudCutoff>0.16</pointCloudCutoff>
+        <pointCloudCutoffMax>10.0</pointCloudCutoffMax>
+      </plugin>
+    </sensor>
+  </gazebo>
 </robot>

Commit message: push

File: src/motoman/motoman_hc10_support/urdf/hc10.xacro (robot description, xacro)
@@ -19,5 +19,7 @@
         <box size="1 0.5 0.05"/>
       </geometry>
-      <material name="Brown"/>
+      <material name="Brown">
+  <color rgba="0.59 0.29 0.0 1.0"/>
+</material>
     </visual>
   </link>
@@ -35,5 +37,5 @@
         <box size="0.05 0.05 0.05"/>
       </geometry>
-      <material name="Gray"/>
+      <material name="Grey"/>
     </visual>
   </link>

File: src/motoman/motoman_hc10_support/urdf/hc10_macro.xacro (robot description, xacro)
@@ -134,8 +134,4 @@
     <!-- end of link list -->
     <!-- joint list -->
-    <joint name="world_prefix" type="fixed">
-      <parent link="world"/>
-      <child link="${prefix}base_link"/>
-    </joint>
     <joint name="${prefix}joint_1_s" type="revolute">
       <parent link="${prefix}base_link"/>
