Commit message: Update hc10_macro.xacro

File: src/motoman/motoman_hc10_support/urdf/hc10_macro.xacro (robot description, xacro)
@@ -199,4 +199,84 @@
       <child link="${prefix}base"/>
     </joint>
+    <xacro:macro name="control" params="joint">
+        <transmission name="${joint}_transmission">
+            <type>transmission_interface/SimpleTransmission</type>
+            <!-- The EffortJointInterface works best with Gazebo using torques to actuate the joints -->
+            <joint name="${joint}">
+                <hardwareInterface>hardware_interface/EffortJointInterface</hardwareInterface>
+            </joint>
+            <actuator name="${joint}_motor">
+                <hardwareInterface>hardware_interface/EffortJointInterface</hardwareInterface>
+                <mechanicalReduction>1</mechanicalReduction>
+            </actuator>
+        </transmission>
+    </xacro:macro>
+    <gazebo>
+      <plugin name="gazebo_ros_control" filename="libgazebo_ros_control.so">
+        <robotNamespace>/${prefix}</robotNamespace>
+        <legacyModeNS>true</legacyModeNS>
+      </plugin>
+    </gazebo>
+	<!-- Transmissions: PositionJointInterface simple -->
+	<transmission name="${prefix}trans_joint_1_s">
+	  <type>transmission_interface/SimpleTransmission</type>
+	  <joint name="${prefix}joint_1_s">
+		<hardwareInterface>hardware_interface/EffortJointInterface</hardwareInterface>
+	  </joint>
+	  <actuator name="${prefix}motor_1_s">
+		<hardwareInterface>hardware_interface/EffortJointInterface</hardwareInterface>
+		<mechanicalReduction>1</mechanicalReduction>
+	  </actuator>
+	</transmission>
+	<transmission name="${prefix}trans_joint_2_l">
+	  <type>transmission_interface/SimpleTransmission</type>
+	  <joint name="${prefix}joint_2_l">
+		<hardwareInterface>hardware_interface/EffortJointInterface</hardwareInterface>
+	  </joint>
+	  <actuator name="${prefix}motor_2_l">
+		<hardwareInterface>hardware_interface/EffortJointInterface</hardwareInterface>
+		<mechanicalReduction>1</mechanicalReduction>
+	  </actuator>
+	</transmission>
+	<transmission name="${prefix}trans_joint_3_u">
+	  <type>transmission_interface/SimpleTransmission</type>
+	  <joint name="${prefix}joint_3_u">
+		<hardwareInterface>hardware_interface/EffortJointInterface</hardwareInterface>
+	  </joint>
+	  <actuator name="${prefix}motor_3_u">
+		<hardwareInterface>hardware_interface/EffortJointInterface</hardwareInterface>
+		<mechanicalReduction>1</mechanicalReduction>
+	  </actuator>
+	</transmission>
+	<transmission name="${prefix}trans_joint_4_r">
+	  <type>transmission_interface/SimpleTransmission</type>
+	  <joint name="${prefix}joint_4_r">
+		<hardwareInterface>hardware_interface/EffortJointInterface</hardwareInterface>
+	  </joint>
+	  <actuator name="${prefix}motor_4_r">
+		<hardwareInterface>hardware_interface/EffortJointInterface</hardwareInterface>
+		<mechanicalReduction>1</mechanicalReduction>
+	  </actuator>
+	</transmission>
+	<transmission name="${prefix}trans_joint_5_b">
+	  <type>transmission_interface/SimpleTransmission</type>
+	  <joint name="${prefix}joint_5_b">
+		<hardwareInterface>hardware_interface/EffortJointInterface</hardwareInterface>
+	  </joint>
+	  <actuator name="${prefix}motor_5_b">
+		<hardwareInterface>hardware_interface/EffortJointInterface</hardwareInterface>
+		<mechanicalReduction>1</mechanicalReduction>
+	  </actuator>
+	</transmission>
+	<transmission name="${prefix}trans_joint_6_t">
+	  <type>transmission_interface/SimpleTransmission</type>
+	  <joint name="${prefix}joint_6_t">
+		<hardwareInterface>hardware_interface/EffortJointInterface</hardwareInterface>
+	  </joint>
+	  <actuator name="${prefix}motor_6_t">
+		<hardwareInterface>hardware_interface/EffortJointInterface</hardwareInterface>
+		<mechanicalReduction>1</mechanicalReduction>
+	  </actuator>
+	</transmission>
   </xacro:macro>
 </robot>

Commit message: push

File: src/motoman/motoman_hc10_support/urdf/hc10_macro.xacro (robot description, xacro)
@@ -132,4 +132,6 @@
     </link>
     <link name="${prefix}tool0"/>
+    <link name="${prefix}camera_link"/>
+    <link name="${prefix}camera_depth_optical_frame"/>
     <!-- end of link list -->
     <!-- joint list -->
@@ -191,5 +193,51 @@
       <child link="${prefix}tool0"/>
     </joint>
+    <joint name="${prefix}camera_joint" type="fixed">
+      <parent link="${prefix}tool0"/>
+      <child link="${prefix}camera_link"/>
+      <origin xyz="0 0 0.1" rpy="0 0 0"/>
+    </joint>
+    <joint name="${prefix}camera_optical_joint" type="fixed">
+      <parent link="${prefix}camera_link"/>
+      <child link="${prefix}camera_depth_optical_frame"/>
+      <origin xyz="0 0 0.1" rpy="0 0 0"/>
+    </joint>
     <!-- end of joint list -->
+    <gazebo reference="${prefix}camera_link">
+  	  <sensor name="kinect_camera" type="depth">
+    	  <update_rate>20</update_rate>
+    	  <camera>
+      	  <horizontal_fov>1.047198</horizontal_fov>
+          <image>
+            <width>640</width>
+            <height>480</height>
+            <format>B8G8R8</format>
+  	      </image>
+          <clip>
+            <near>0.05</near>
+            <far>3</far>
+          </clip>
+        </camera>
+        <plugin name="kinect_controller" filename="libgazebo_ros_openni_kinect.so">
+        <baseline>0.1</baseline>
+        <alwaysOn>true</alwaysOn>
+        <updateRate>10</updateRate>
+        <cameraName>camera_ir</cameraName>
+        <imageTopicName>/camera/color/image_raw</imageTopicName>
+        <cameraInfoTopicName>/camera/color/camera_info</cameraInfoTopicName>
+        <depthImageTopicName>/camera/depth/image_raw</depthImageTopicName>
+        <depthImageCameraInfoTopicName>/camera/depth/camera_info</depthImageCameraInfoTopicName>
+        <pointCloudTopicName>/camera/depth/points</pointCloudTopicName>
+        <frameName>camera_depth_optical_frame</frameName>
+        <distortion_k1>0.0</distortion_k1>
+        <distortion_k2>0.0</distortion_k2>
+        <distortion_k3>0.0</distortion_k3>
+        <distortion_t1>0.0</distortion_t1>
+        <distortion_t2>0.0</distortion_t2>
+        <pointCloudCutoff>0.16</pointCloudCutoff>
+        <pointCloudCutoffMax>10.0</pointCloudCutoffMax>
+        </plugin>
+      </sensor>
+    </gazebo>
     <!-- ROS base_link to Robot Manufacturer World Coordinates transform -->
     <link name="${prefix}base" />

Commit message: commit final

File: src/motoman/motoman_hc10_support/urdf/hc10_macro.xacro (robot description, xacro)
@@ -196,5 +196,5 @@
       <parent link="${prefix}tool0"/>
       <child link="${prefix}camera_link"/>
-      <origin xyz="0 0 0.1" rpy="0 0 0"/>
+      <origin xyz="0 0 0.1" rpy="0 -1.57 3.14"/>
     </joint>
     <joint name="${prefix}camera_optical_joint" type="fixed">
